File: Hardware/ldo.kicad_sch (KiCad schematic)
At the start: 23 parts, among them IC1 TPS61089RNRR, IC2 AP2205-W5-7

Commit message: 2nd review of schematic
Parts:
- added C53: 1uF, Capacitor_SMD:C_0402_1005Metric, symbol Device:C_Small
- added C54, C62: 10uF, Capacitor_SMD:C_0603_1608Metric, symbol Device:C_Small
- added C55: 120pF, Capacitor_SMD:C_0402_1005Metric, symbol Device:C_Small
- added C56: 2.2nF, Capacitor_SMD:C_0402_1005Metric, symbol Device:C_Small
- added C57, C59: 22uF, Capacitor_SMD:C_0805_2012Metric, symbol Device:C_Small
- added C58: 2.2uF, Capacitor_SMD:C_0402_1005Metric, symbol Device:C_Small
- added C60, C61, C63: 100nF, Capacitor_SMD:C_0402_1005Metric, symbol Device:C_Small
- added C64: 22uF, Capacitor_SMD:C_1206_3216Metric, symbol Device:C_Small
- added IC4: AP2205-W5-7, iclr:SOT95P282X145-5N, symbol iclr:AP2205-W5-7
- added IC5: TPS61089RNRR, iclr:IC_TPS61089RNRR, symbol iclr:TPS61089RNRR
- added L5: SRR6038-5R0Y, iclr:IND_SRP6540-390M, symbol iclr:SRR6038-5R0Y
- added R51: 18.7k, Resistor_SMD:R_0402_1005Metric, symbol Device:R_Small
- added R52: 976k, Resistor_SMD:R_0402_1005Metric, symbol Device:R_Small
- added R53: 100k, Resistor_SMD:R_0402_1005Metric, symbol Device:R_Small
- added R54: 49.9k, Resistor_SMD:R_0402_1005Metric, symbol Device:R_Small
- added R55: 432k, Resistor_SMD:R_0402_1005Metric, symbol Device:R_Small
- added R56: 10K, Resistor_SMD:R_0402_1005Metric, symbol Device:R_Small
- added R57: 475k, Resistor_SMD:R_0402_1005Metric, symbol Device:R_Small
- added R58: 287k, Resistor_SMD:R_0402_1005Metric, symbol Device:R_Small
- renumbered C32 to C41, C33 to C42, C34 to C43, C35 to C44, C36 to C45, C37 to C46, C38 to C47, C39 to C48, C40 to C49, C41 to C50, C42 to C51, C43 to C52, IC1 to IC2, IC2 to IC3, R34 to R43, R36 to R44, R38 to R45, R40 to R46, R42 to R47, R43 to R48, R44 to R49, R45 to R50
Connections:
- net +3V3: now also C61.1, C64.1, IC5.9 (VIN), L5.1, R56.2
- net GND: now also C53.2, C54.2, C55.2, C56.2, C57.2, C58.2, C59.2, C61.2, C62.2, C63.2, C64.2, IC4.2 (GND), IC5.5 (GND), R53.1, R54.1, R57.1
- new net: C56.1, R51.2
- new net: C55.1, IC5.4 (COMP), R51.1
- new net: IC5.8 (ILIM), R57.2
- new net: C60.1, IC5.10 (BOOT)
- new net: C60.2, IC5.11 (SW), L5.2, R58.2
- new net: C54.1, IC5.2 (VCC)
- new net: IC5.7 (EN), R56.1
- new net: IC4.4 (ADJ/NC), R54.2, R55.1
- new net 12V: C58.1, IC4.5 (VOUT), R55.2
- new net FB_12V: IC5.3 (FB), R52.1, R53.2
- new net LDO12V_IN: C53.1, C57.1, C59.1, C62.1, C63.1, IC4.1 (VIN), IC4.3 (EN), IC5.6 (VOUT), R52.2
- new net SW_12V: IC5.1 (FSW), R58.1
Other:
- note added: "SIM: https://webench.ti.com/appinfo/webench/scripts/SDP.cgi?ID=0086ECB0F8B2BBA7"
- note added: "SIM: https://webench.ti.com/appinfo/webench/scripts/SDP.cgi?ID=C25BB1AA15C31C1A"
- moved on the sheet: C41, C42, C43, C44, C45, C46, C47, C48, C49, C50, C51, C52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
