File: Hardware/buck.kicad_sch (KiCad schematic)
At the start: 30 parts, among them Q1 SSM3K15AMFV,L3F, U8 SiC437AED-T1

Commit message: 2nd review of schematic
Parts:
- renumbered C44 to C65, C45 to C66, C46 to C67, C47 to C68, C48 to C69, C49 to C70, C58 to C71, C49 to C72, C47 to C73, C59 to C74, C60 to C75, C61 to C76, C62 to C77, C46 to C78, C48 to C79, C64 to C80, C65 to C81, L5 to L6, R46 to R59, R47 to R60, R48 to R61, R49 to R62, R52 to R63, R53 to R64, R54 to R65, R55 to R66, R56 to R67, R59 to R68

Commit message: pcb and schematic update
Found all footprints including J3, pressure controller, tvs diode. PCB infrastructure update
Other:
- note added: "Vref = 0.6V The resistor pair here to boost the voltage to 6V or 7.38V"
Changed lines of the file:
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@@
+		)
+	)
+	(text "Vref = 0.6V\nThe resistor pair here to boost the voltage to 6V or 7.38V"
+		(exclude_from_sim no)
+		(at 136.906 48.514 0)
+		(effects
+			(font
+				(size 1.27 1.27)
+			)
 		)
 	)
@@
 		)
 	)
-	(text_box "Remove this resistor for 8.4V mode"
+	(text_box "Remove this resistor for 7.4V mode"
 		(exclude_from_sim no)
 		(at 132.08 52.07 0)
@@
 		(stroke
 			(width -0.0001)
-			(type default)
+			(type solid)
 		)
 		(fill
