File: Hardware/power.kicad_sch (KiCad schematic)
At the start: 20 parts, among them U3 LM66200DRLR, U4 MAX77827AEFD+T, U5 SC4215ASTRT

Commit message: 2nd review of schematic
Parts:
- renumbered C20 to C17, C21 to C18, C22 to C19, C23 to C20, C24 to C21, C25 to C22, C26 to C23, C27 to C24, R14 to R16, R15 to R17, R16 to R18, R17 to R19, TP4 to TP5, TP5 to TP6, TP6 to TP7
