File: Hardware/thermocouple.kicad_sch (KiCad schematic)
At the start: 18 parts, among them U6 MAX31856, U7 MAX31856

Commit message: 2nd review of schematic
Parts:
- renumbered C53 to C31, C54 to C32, C55 to C33, C56 to C34, C57 to C35, C19 to C36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
Connections:
- net CS renamed CS0
- net CS0: no longer U6.9 (~{CS})
- net DRDY renamed DRDY0
- net DRDY0: no longer U6.7 (~{DRDY})
- net FAULT renamed FAULT0
- net FAULT0: no longer U6.13 (~{FAULT})
- new net CS1: U6.9 (~{CS})
- new net DRDY1: U6.7 (~{DRDY})
- new net FAULT1: U6.13 (~{FAULT})
