File: Hardware/thermocouple.kicad_sch (KiCad schematic)
At the start: 18 parts, among them U6 MAX31856, U7 MAX31856

Commit message: tiny tweaks and ready to order
Parts:
- C901: renamed from C31; value 0.01uF -> 10nF
- C902: renamed from C32; value 0.1uF -> 100nF
- C903: renamed from C33; value 0.01uF -> 10nF
- C904: renamed from C34; value 0.1uF -> 100nF
- C905: renamed from C35; value 0.1uF -> 100nF
- C906: renamed from C36; value 0.01uF -> 10nF
- C907: renamed from C37; value 0.1uF -> 100nF
- C908: renamed from C38; value 0.01uF -> 10nF
- C909: renamed from C39; value 0.1uF -> 100nF
- C910: renamed from C40; value 0.1uF -> 100nF
- J901: renamed from TC1; value Thermocouple -> 1053131102
- J902: renamed from TC2; value Thermocouple -> 1053131102
- R901: renamed from R39; value 100 -> 100Ω
- R902: renamed from R40; value 100 -> 100Ω
- R903: renamed from R41; value 100 -> 100Ω
- R904: renamed from R42; value 100 -> 100Ω
- renumbered U6 to U901, U7 to U902
