File: Hardware/pressure.kicad_sch (KiCad schematic)
At the start: 44 parts, among them IC3 ADS131M03IRUKR, IC5 ADS131M04IRUKR, J4 1053131104, J5 1053131104, J6 1053131104

Commit message: Updated connections
Parts:
- removed IC3: ADS131M03IRUKR, QFN40P300X300X80-21N-D, symbol ADS131M03IRUKR:ADS131M03IRUKR
Changed lines of the file:
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@@
-	)
-	(symbol
-		(lib_id "ADS131M03IRUKR:ADS131M03IRUKR")
-		(at 29.21 140.97 0)
-		(unit 1)
-		(exclude_from_sim no)
-		(in_bom yes)
-		(on_board yes)
-		(dnp no)
-		(fields_autoplaced yes)
-		(property "Reference" "IC3"
-			(at 64.77 134.5498 0)
-			(effects
-				(font
-					(size 1.27 1.27)
-				)
-			)
-		)
-		(property "Value" "ADS131M03IRUKR"
-			(at 64.77 137.0898 0)
-			(effects
-				(font
-					(size 1.27 1.27)
-				)
-			)
-		)
-		(property "Footprint" "QFN40P300X300X80-21N-D"
-			(at 55.88 225.73 0)
-			(effects
-				(font
-					(size 1.27 1.27)
-				)
-				(justify left top)
-				(hide yes)
-			)
-		)
-		(property "Datasheet" "https://www.ti.com/general/docs/suppproductinfo.tsp?distId=10&gotoUrl=http%3A%2F%2Fwww.ti.com%2Flit%2Fgpn%2Fads131m03"
-			(at 55.88 325.73 0)
-			(effects
-				(font
-					(size 1.27 1.27)
-				)
-				(justify left top)
-				(hide yes)
-			)
-		)
-		(property "Description" "Encoders, Decoders, Multiplexers & Demultiplexers 24-bit, 32-kSPS, 3-channel, simultaneous-sampling, delta-sigma ADC 20-WQFN -40 to 125"
-			(at 29.21 140.97 0)
-			(effects
-				(font
-					(size 1.27 1.27)
-				)
-				(hide yes)
-			)
-		)
-		(property "Height" "0.8"
-			(at 55.88 525.73 0)
-			(effects
-				(font
-					(size 1.27 1.27)
-				)
-				(justify left top)
-				(hide yes)
-			)
-		)
-		(property "Mouser Part Number" "595-ADS131M03IRUKR"
-			(at 55.88 625.73 0)
-			(effects
-				(font
-					(size 1.27 1.27)
-				)
-				(justify left top)
-				(hide yes)
-			)
-		)
-		(property "Mouser Price/Stock" "https://www.mouser.co.uk/ProductDetail/Texas-Instruments/ADS131M03IRUKR?qs=stqOd1AaK7%252Bm3QT30xDCgA%3D%3D"
-			(at 55.88 725.73 0)
-			(effects
-				(font
-					(size 1.27 1.27)
-				)
-				(justify left top)
-				(hide yes)
-			)
-		)
-		(property "Manufacturer_Name" "Texas Instruments"
-			(at 55.88 825.73 0)
-			(effects
-				(font
-					(size 1.27 1.27)
-				)
-				(justify left top)
-				(hide yes)
-			)
-		)
-		(property "Manufacturer_Part_Number" "ADS131M03IRUKR"
-			(at 55.88 925.73 0)
-			(effects
-				(font
-					(size 1.27 1.27)
-				)
-				(justify left top)
-				(hide yes)
-			)
-		)
-		(pin "1"
-		)
-		(pin "6"
-		)
-		(pin "18"
-		)
-		(pin "9"
-		)
-		(pin "14"
-		)
-		(pin "13"
-		)
-		(pin "2"
-		)
-		(pin "17"
-		)
-		(pin "15"
-		)
-		(pin "3"
-		)
-		(pin "4"
-		)
-		(pin "16"
-		)
-		(pin "11"
-		)
-		(pin "21"
-		)
-		(pin "5"
-		)
-		(pin "7"
-		)
-		(pin "20"
-		)
-		(pin "19"
-		)
-		(pin "8"
-		)
-		(pin "10"
-		)
-		(pin "12"
-		)
-		(instances
-			(project ""
-				(path "/7db990e4-92e1-4f99-b4d2-435bbec1ba83/3af81d2a-0ad1-4f51-8454-076646dec8d9"
-					(reference "IC3")
-					(unit 1)
-				)
-			)
-		)
 	)
 	(symbol

Commit message: 2nd review of schematic
Parts:
- removed JP11, JP16, JP8: SolderJumper_2_Open, iclr:SmallerSolderJP, symbol Jumper:SolderJumper_2_Open
- renumbered C50 to C25, C51 to C26, C52 to C27, C63 to C28, C18 to C29, C12 to C30, IC5 to IC1, J5 to J4, J6 to J5, J4 to J6, JP17 to JP11, JP4 to JP12, JP7 to JP13, JP9 to JP14, JP12 to JP15, JP6 to JP4, JP13 to JP5, JP5 to JP6, JP14 to JP7, JP19 to JP8, JP15 to JP9, R35 to R21, R39 to R22, R37 to R23, R26 to R24, R27 to R25, R28 to R26, R57 to R27, R29 to R28, R41 to R29, R58 to R31, R31 to R32, R20 to R33, R21 to R34, R22 to R35, R23 to R36, R24 to R37, R25 to R38
Connections:
- net AIN0N: no longer C29.2, C30.2, R32.2, R38.2
- net AIN0P: no longer C29.1, C30.1, R28.2, R36.2
- net AIN1N: now also C30.2, R38.2
- net AIN1P: now also C30.1, R36.2
- net AIN2N: now also C29.2, R32.2
- net AIN2P: now also C29.1, R28.2
- net GND: now also J4.3, J5.3, J6.3, R29.2, R30.2, R31.1, R32.1, R37.2, R38.1
- net AIN3N: no longer names the net of IC1.7 (AIN3N)
- net AIN3P: no longer names the net of IC1.8 (AIN3P)
- no-connect marks 0 -> 2
Other:
- note added: "10V"
- note removed: "12V"
- note removed: "Jump for voltage"
- moved on the sheet: C25, C26, C27, IC1

Commit message: pcb and schematic update
Found all footprints including J3, pressure controller, tvs diode. PCB infrastructure update
Parts:
- IC1: footprint QFN40P300X300X80-21N-D -> iclr:QFN40P300X300X80-21N-D
Changed lines of the file:
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@@
 			)
 		)
-		(property "Footprint" "QFN40P300X300X80-21N-D"
+		(property "Footprint" "iclr:QFN40P300X300X80-21N-D"
 			(at 163.5 95.25 0)
 			(effects

Commit message: Routing Improvement
Version 3. Mainly solved 3 problem: 1. clock and decoupler closer to microcontroller; 2. Route of Data+ and Data- neater; 3. wider trace for 6v and 16.8v
Parts:
- J4, J5, J6: footprint Connector_Molex:Molex_Nano-Fit_105313-xx04_1x04_P2.50mm_Horizontal -> Connector_Molex:Molex_Nano-Fit_105313-xx03_1x03_P2.50mm_Horizontal; symbol iclr:1053131104 -> Connector:Conn_01x03_Pin
Connections:
- net GND: no longer J4.4, J5.4, J6.4
