File: Hardware/pressure.kicad_sch (KiCad schematic)
At the start: 40 parts, among them IC1 ADS131M04IRUKR, J4 1053131104, J5 1053131104, J6 1053131104

Commit message: Version 5
Parts:
- added C83, C84, C85: 100nF, Capacitor_SMD:C_0402_1005Metric, symbol Device:C
Connections:
- net GND: now also C83.1, C84.1, C85.1
- net at J5.1 (Pin_1), JP11.2 (C): now also C85.2
- net at J6.1 (Pin_1), JP15.2 (C): now also C84.2
- net at J4.1 (Pin_1), JP10.2 (C): now also C83.2
Other:
- moved on the sheet: JP10, JP11, JP15

Commit message: tiny tweaks and ready to order
Parts:
- J801: renamed from J4; value 1053131104 -> 1053131103
- J802: renamed from J5; value 1053131104 -> 1053131103
- J803: renamed from J6; value 1053131104 -> 1053131103
- JP801: renamed from JP4; now left out of the parts list
- JP802: renamed from JP5; now left out of the parts list
- JP803: renamed from JP6; now left out of the parts list
- JP804: renamed from JP7; now left out of the parts list
- JP805: renamed from JP8; now left out of the parts list
- JP806: renamed from JP9; now left out of the parts list
- JP807: renamed from JP10; now left out of the parts list
- JP808: renamed from JP11; now left out of the parts list
- JP809: renamed from JP12; now left out of the parts list
- JP810: renamed from JP13; now left out of the parts list
- JP811: renamed from JP14; now left out of the parts list
- JP812: renamed from JP15; now left out of the parts list
- R801: renamed from R21; value 75k -> 75kΩ
- R802: renamed from R22; value 14k -> 14kΩ
- R803: renamed from R23; value 10k -> 10kΩ
- R804: renamed from R24; value 75k -> 75kΩ
- R805: renamed from R25; value 14k -> 14kΩ
- R806: renamed from R26; value 10k -> 10kΩ
- R807: renamed from R27; value 1k -> 1kΩ
- R808: renamed from R28; value 1k -> 1kΩ
- R809: renamed from R29; value 49.9 -> 49.9Ω
- R810: renamed from R30; value 49.9 -> 49.9Ω
- R811: renamed from R31; value 1k -> 1kΩ
- R812: renamed from R32; value 1k -> 1kΩ
- R813: renamed from R33; value 75k -> 75kΩ
- R814: renamed from R34; value 14k -> 14kΩ
- R815: renamed from R35; value 10k -> 10kΩ
- R816: renamed from R36; value 1k -> 1kΩ
- R817: renamed from R37; value 49.9 -> 49.9Ω
- R818: renamed from R38; value 1k -> 1kΩ
- renumbered C25 to C801, C26 to C802, C27 to C803, C28 to C804, C29 to C805, C83 to C806, C85 to C807, C30 to C808, C84 to C809, IC1 to U801
