File: Hardware/Reggie.kicad_sch (KiCad schematic)
At the start: 40 parts, among them J1 RBUS, U1 ESP32-S3, Y1 R940000171

Commit message: Overall Packing Backup Version
Connections:
- net GPIO13: now reaches U1.18 (GPIO13/ADC2_CH2)
- net GPIO14: now reaches U1.19 (GPIO14/ADC2_CH3)
- net GPIO15: now reaches U1.21 (GPIO15/ADC2_CH4/XTAL_32K_P)
- net GPIO16: now reaches U1.22 (GPIO16/ADC2_CH5/XTAL_32K_N)
- net GPIO39: now reaches U1.44 (MTCK/JTAG/GPIO39)
- net GPIO4: now reaches U1.9 (GPIO4/ADC1_CH3)
- no-connect marks 11 -> 15
Other:
- added sheet GPIO tvs (GPIO_Breakout.kicad_sch)
- sheet Servo ports: added ServoPWM; removed none

Commit message: Overall Routing Complete!!!
Version2
Connections:
- net GPIO1: now reaches U1.6 (GPIO1/ADC1_CH0)
- net GPIO2: now reaches U1.7 (GPIO2/ADC1_CH1)
- net GPIO16: no longer names the net of U1.22 (GPIO16/ADC2_CH5/XTAL_32K_N)
- net GPIO39: no longer names the net of U1.44 (MTCK/JTAG/GPIO39)
Other:
- sheet GPIO tvs ports: added GPIO1, GPIO2; removed GPIO16, GPIO39
Changed lines of the file:
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@@
 	)
 	(no_connect
-		(at 69.85 74.93)
-	)
-	(no_connect
 		(at 135.89 77.47)
 	)
@@
 	)
 	(no_connect
+		(at 69.85 118.11)
+	)
+	(no_connect
 		(at 135.89 85.09)
 	)
@@
 	)
 	(no_connect
-		(at 69.85 72.39)
-	)
-	(no_connect
 		(at 69.85 62.23)
 	)
@@
 	)
 	(no_connect
+		(at 135.89 130.81)
+	)
+	(no_connect
 		(at 135.89 82.55)
 	)
@@
 	(wire
 		(pts
+			(xy 58.42 72.39) (xy 69.85 72.39)
+		)
+		(stroke
+			(width 0)
+			(type default)
+		)
+	)
+	(wire
+		(pts
 			(xy 62.23 95.25) (xy 69.85 95.25)
 		)
@@
 		)
 	)
-	(wire
-		(pts
-			(xy 54.61 118.11) (xy 69.85 118.11)
-		)
-		(stroke
-			(width 0)
-			(type default)
-		)
-	)
 	(polyline
 		(pts
@@
 	(wire
 		(pts
+			(xy 58.42 74.93) (xy 69.85 74.93)
+		)
+		(stroke
+			(width 0)
+			(type default)
+		)
+	)
+	(wire
+		(pts
 			(xy 167.64 127) (xy 167.64 132.08)
 		)
@@
 		)
 	)
-	(label "GPIO16"
-		(at 135.89 130.81 0)
-		(effects
-			(font
-				(size 1.27 1.27)
-			)
-			(justify left bottom)
-		)
-	)
 	(label "VSPI_MISO"
 		(at 139.7 107.95 0)
@@
 		)
 	)
-	(label "GPIO39"
-		(at 54.61 118.11 180)
+	(label "GPIO1"
+		(at 58.42 72.39 180)
 		(effects
 			(font
@@
 		)
 	)
+	(label "GPIO2"
+		(at 58.42 74.93 180)
+		(effects
+			(font
+				(size 1.27 1.27)
+			)
+			(justify right bottom)
+		)
+	)
 	(label "HSPI_SCLK"
 		(at 139.7 100.33 0)
@@
 		)
 	)
-	(label "GPIO16"
+	(label "GPIO2"
 		(at 240.03 105.41 180)
 		(effects
@@
 		)
 	)
-	(label "GPIO39"
+	(label "GPIO1"
 		(at 240.03 107.95 180)
 		(effects
@@
 			)
 		)
-		(pin "GPIO16" bidirectional
+		(pin "GPIO2" bidirectional
 			(at 243.84 105.41 180)
 			(effects
@@
 			)
 		)
-		(pin "GPIO39" bidirectional
+		(pin "GPIO1" bidirectional
 			(at 243.84 107.95 180)
 			(effects

Commit message: Filled zones and via location
Version 4. allocate filled zones and vias, also reassigned pins from microcontroller
Connections:
- net GPIO2 is gone; now on net ServoPWM: U1.7 (GPIO2/ADC1_CH1)
- net GPIO4 is gone; now on net ADS_CLK: U1.9 (GPIO4/ADC1_CH3)
- net ADS_CLK: no longer U1.11 (GPIO6/ADC1_CH5)
- net ADS_CS: now also U1.11 (GPIO6/ADC1_CH5); no longer U1.23 (GPIO17/ADC2_CH6/DAC_2)
- net BUCK_EN: now also U1.27 (GPIO21); no longer U1.37 (SPICLK_P/GPIO47)
- net SD_CS: now also U1.41 (GPIO36); no longer U1.17 (GPIO12/ADC2_CH1)
- net SD_DET: now also U1.49 (U0TXD/PROG/GPIO43); no longer U1.16 (GPIO11/ADC2_CH0)
- net SD_EN: now also U1.48 (MTMS/JTAG/GPIO42); no longer U1.15 (GPIO10/ADC1_CH9)
- net ServoPWM: no longer U1.14 (GPIO9/ADC1_CH8)
- net T_CS0: now also U1.12 (GPIO7/ADC1_CH6); no longer U1.27 (GPIO21)
- net T_CS1: now also U1.14 (GPIO9/ADC1_CH8); no longer U1.45 (MTDO/JTAG/GPIO40)
- net T_DRDY0: now also U1.17 (GPIO12/ADC2_CH1); no longer U1.13 (GPIO8/ADC1_CH7)
- net T_DRDY1: now also U1.16 (GPIO11/ADC2_CH0); no longer U1.48 (MTMS/JTAG/GPIO42)
- net T_FAULT0: now also U1.13 (GPIO8/ADC1_CH7); no longer U1.12 (GPIO7/ADC1_CH6)
- net T_FAULT1: now also U1.15 (GPIO10/ADC1_CH9); no longer U1.47 (MTDI/JTAG/GPIO41)
- net VSPI_MISO: now also U1.47 (MTDI/JTAG/GPIO41); no longer U1.43 (GPIO38)
- net VSPI_MOSI: now also U1.42 (GPIO37); no longer U1.41 (GPIO36)
- net VSPI_SCLK: now also U1.43 (GPIO38); no longer U1.42 (GPIO37)
- net TVS3: now reaches U1.22 (GPIO16/ADC2_CH5/XTAL_32K_N)
- net TVS4: now reaches U1.24 (GPIO18/ADC2_CH7/DAC_1)
- net at R7.2: now also U1.37 (SPICLK_P/GPIO47); no longer U1.49 (U0TXD/PROG/GPIO43)
- net GPIO1: no longer names the net of U1.6 (GPIO1/ADC1_CH0)
- net GPIO13 renamed TVS1
- net GPIO14 renamed TVS5
- net GPIO15 renamed TVS6
- new net TVS7: U1.23 (GPIO17/ADC2_CH6/DAC_2)
Other:
- sheet GPIO tvs ports: added TVS1, TVS3, TVS4, TVS5, TVS6, TVS7; removed GPIO1, GPIO13, GPIO14, GPIO15, GPIO2, GPIO4
- moved on the sheet: R7
