File: Hardware/GPIO_Breakout.kicad_sch (KiCad schematic)
At the start: 2 parts, among them J8 GPIO Breakout

Commit message: tiny tweaks and ready to order
Parts:
- J1001: renamed from J8; now left out of the parts list
- renumbered D6 to D1001
Changed lines of the file:
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@@
 		(dnp no)
 		(fields_autoplaced yes)
-		(property "Reference" "#PWR0151"
+		(property "Reference" "#PWR01002"
 			(at 107.95 39.37 0)
 			(effects
@@
 		)
 		(instances
-			(project "Reggie"
-				(path "/7db990e4-92e1-4f99-b4d2-435bbec1ba83/27542141-17da-4259-86dc-4e9093aea81a"
-					(reference "#PWR0151")
+			(project "Heimdall"
+				(path "/7db990e4-92e1-4f99-b4d2-435bbec1ba83/27542141-17da-4259-86dc-4e9093aea81a"
+					(reference "#PWR01002")
 					(unit 1)
 				)
@@
 		(unit 1)
 		(exclude_from_sim no)
-		(in_bom yes)
+		(in_bom no)
 		(on_board yes)
 		(dnp no)
-		(property "Reference" "J8"
-			(at 121.92 53.34 90)
+		(property "Reference" "J1001"
+			(at 122.428 46.7391 0)
 			(effects
 				(font
@@
 		)
 		(property "Value" "GPIO Breakout"
-			(at 124.4569 53.34 90)
+			(at 122.428 49.276 0)
 			(effects
 				(font
@@
 		)
 		(instances
-			(project "Reggie"
-				(path "/7db990e4-92e1-4f99-b4d2-435bbec1ba83/27542141-17da-4259-86dc-4e9093aea81a"
-					(reference "J8")
+			(project "Heimdall"
+				(path "/7db990e4-92e1-4f99-b4d2-435bbec1ba83/27542141-17da-4259-86dc-4e9093aea81a"
+					(reference "J1001")
 					(unit 1)
 				)
@@
 		(dnp no)
 		(fields_autoplaced yes)
-		(property "Reference" "D6"
+		(property "Reference" "D1001"
 			(at 67.31 39.37 0)
 			(effects
@@
 		)
 		(instances
-			(project "Reggie"
-				(path "/7db990e4-92e1-4f99-b4d2-435bbec1ba83/27542141-17da-4259-86dc-4e9093aea81a"
-					(reference "D6")
+			(project "Heimdall"
+				(path "/7db990e4-92e1-4f99-b4d2-435bbec1ba83/27542141-17da-4259-86dc-4e9093aea81a"
+					(reference "D1001")
 					(unit 1)
 				)
@@
 		(dnp no)
 		(fields_autoplaced yes)
-		(property "Reference" "#PWR0150"
+		(property "Reference" "#PWR01001"
 			(at 41.91 55.88 0)
 			(effects
@@
 		)
 		(instances
-			(project "Reggie"
-				(path "/7db990e4-92e1-4f99-b4d2-435bbec1ba83/27542141-17da-4259-86dc-4e9093aea81a"
-					(reference "#PWR0150")
+			(project "Heimdall"
+				(path "/7db990e4-92e1-4f99-b4d2-435bbec1ba83/27542141-17da-4259-86dc-4e9093aea81a"
+					(reference "#PWR01001")
 					(unit 1)
 				)
@@
 		(dnp no)
 		(fields_autoplaced yes)
-		(property "Reference" "#PWR0152"
+		(property "Reference" "#PWR01003"
 			(at 118.11 49.53 0)
 			(effects
@@
 		)
 		(instances
-			(project "Reggie"
-				(path "/7db990e4-92e1-4f99-b4d2-435bbec1ba83/27542141-17da-4259-86dc-4e9093aea81a"
-					(reference "#PWR0152")
-					(unit 1)
-				)
+			(project "Heimdall"
+				(path "/7db990e4-92e1-4f99-b4d2-435bbec1ba83/27542141-17da-4259-86dc-4e9093aea81a"
+					(reference "#PWR01003")
+					(unit 1)
+				)
