File: Hardware/Heimdall.kicad_pcb (KiCad board)
At the start: 4 copper layers, 70 x 50 mm, 225 parts, among them IC1 ADS131M04IRUKR, IC2 TPS61089RNRR, IC3 AP2205-W5-7, IC4 AP2205-W5-7, IC5 TPS61089RNRR, J1 RBUS, J2 USB_C_Receptacle_USB2.0, J3 ServoConnector1, J4 1053131104, J5 1053131104, J6 1053131104, J7 ST1W008S4TR2000, J8 GPIO Breakout, Q1 SSM3K15AMFV,L3F, Q2 PMOS, U1 ESP32-S3, U2 SN65HVD230, U3 LM66200DRLR, U4 MAX77827AEFD+T, U5 SC4215ASTRT, U6 MAX31856, U7 MAX31856, U8 SiC437AED-T1, Y1 R940000171

Commit message: Version 5
Parts:
- added C83: 100nF, Capacitor_SMD:C_0402_1005Metric, F.Cu at (183.4, 97.6)
- added C84: 100nF, Capacitor_SMD:C_0402_1005Metric, F.Cu at (183.4, 87.3)
- added C85: 100nF, Capacitor_SMD:C_0402_1005Metric, F.Cu at (183.4, 76.3)
- moved R8 51.3 mm to (183.6, 70.5), turned to 180 degrees
- moved LED5 48.0 mm to (181.8, 70.5), turned to 0 degrees
- moved TP1 12.9 mm to (146.0, 88.3)
- moved R7 12.3 mm to (146.0, 86.3)
- moved LED1 11.3 mm to (146.0, 90.3)
- moved R2 11.3 mm to (146.0, 92.2)
- moved C53 10.4 mm to (178.9, 73.8)
- moved C50 10.3 mm to (167.4, 108.1), turned to 0 degrees
- moved C64 8.57 mm to (172.2, 90.0)
- moved JP1 5.97 mm to (160.9, 86.4), turned to 0 degrees
- moved JP2 4.93 mm to (163.7, 81.4)
- moved R9 2.55 mm to (132.0, 85.9), turned to 90 degrees
- moved C3 2.36 mm to (160.9, 84.1), turned to 0 degrees
- moved C16 2.35 mm to (136.6, 81.1)
- moved C54 2.31 mm to (170.6, 87.3)
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Connections:
- R7 pad 2: Net-(U1-SPICLK_P/GPIO47) -> Net-(U1-U0TXD/PROG/GPIO43)
- U1 pad 10: /ADS_DRDY -> /HSPI_MISO
- U1 pad 11: /ADS_CS -> /HSPI_SCLK
- U1 pad 37: Net-(U1-SPICLK_P/GPIO47) -> /CAN_TX
- U1 pad 38: /HSPI_MOSI -> /CAN_RX
- U1 pad 39: /HSPI_MISO -> /ServoPWM
- U1 pad 40: /HSPI_SCLK -> /SD_DET
- U1 pad 49: /SD_DET -> Net-(U1-U0TXD/PROG/GPIO43)
- U1 pad 51: unconnected-(U1-GPIO45-Pad51) -> /ADS_CLK
- U1 pad 6: unconnected-(U1-GPIO1/ADC1_CH0-Pad6) -> /ADS_DRDY
- U1 pad 7: /ServoPWM -> /ADS_CS
- U1 pad 9: /ADS_CLK -> /HSPI_MOSI
Routing:
- net +12V: track 99.2 -> 37.8 mm, vias 5 -> 4
- net /HSPI_MOSI: track 61.9 -> 43.5 mm, vias 4 -> 3
- net +3V3: track 60.3 -> 42.7 mm, vias 24 -> 29
- net Net-(U1-SPICLK_P/GPIO47): track 17.3 -> 0.00 mm
- net /HSPI_MISO: track 60.1 -> 43.3 mm, vias 4 -> 3
- net /CAN_TX: track 2.08 -> 18.7 mm
- net /HSPI_SCLK: track 58.7 -> 42.3 mm, vias 4 -> 3
- net VBUS: track 58.9 -> 44.5 mm
- net /CAN_RX: track 1.86 -> 14.3 mm
- net /ServoPWM: track 58.9 -> 46.7 mm
- net Net-(IC2-SW): track 9.11 -> 0.26 mm
- net /SD_DET: track 38.8 -> 30.1 mm, vias 3 -> 2
- net Net-(IC5-SW): track 7.98 -> 0.20 mm
- net Net-(U1-U0TXD/PROG/GPIO43): track 0.00 -> 7.43 mm, vias 0 -> 2
- net /CAN-: track 17.0 -> 11.2 mm
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- added copper zone on B.Cu, net +3V3
- added copper zone on B.Cu, net Net-(IC2-SW)
- added copper zone on F.Cu, net Net-(IC2-SW)
- added copper zone on F.Cu, net Net-(IC5-SW)
- removed copper zone on F.Cu, net /TXD

Commit message: tiny tweaks and ready to order
Parts:
- removed R20: 165, Resistor_SMD:R_0402_1005Metric
- C103: renamed from C3; value 0.1uF -> 100nF
- C105: renamed from C5; value 0.1uF -> 100nF
- C106: renamed from C6; value 0.1uF -> 100nF
- C108: renamed from C8; value 0.1uF -> 100nF
- C110: renamed from C10; value 0.1uF -> 100nF
- C111: renamed from C11; value 0.1uF -> 100nF
- C208: renamed from C24; value 0.1uF -> 100nF
- C310: renamed from C74; value 0.1uF -> 100nF
- C701: renamed from C82; value 0.1uF -> 100nF
- C901: renamed from C31; value 0.01uF -> 10nF
- C902: renamed from C32; value 0.1uF -> 100nF
- C903: renamed from C33; value 0.01uF -> 10nF
- C904: renamed from C34; value 0.1uF -> 100nF
- C905: renamed from C35; value 0.1uF -> 100nF
- C906: renamed from C36; value 0.01uF -> 10nF
- C907: renamed from C37; value 0.1uF -> 100nF
- C908: renamed from C38; value 0.01uF -> 10nF
- C909: renamed from C39; value 0.1uF -> 100nF
- C910: renamed from C40; value 0.1uF -> 100nF
- D101: renamed from LED1; value GREEN_LED -> LED_GREEN
- D102: renamed from LED2; value GREEN_LED -> LED_GREEN
- D103: renamed from LED3; value ORANGE_LED -> LED_ORANGE
- D104: renamed from LED4; value BLUE_LED -> LED_BLUE
- D105: renamed from LED5; value RED_LED -> LED_RED
- D602: renamed from LED6; value WHITE_LED -> LED_WHITE
- J1101: renamed from J3; value ServoConnector1 -> 1053131103
- J801: renamed from J4; value 1053131104 -> 1053131103
- J802: renamed from J5; value 1053131104 -> 1053131103
- J803: renamed from J6; value 1053131104 -> 1053131103
- J901: renamed from TC1; value Thermocouple -> 1053131102
- J902: renamed from TC2; value Thermocouple -> 1053131102
- L101: renamed from L1; value 2.0nH -> 2nH
- L401: renamed from L4; value SRR6038-5R0Y -> 5uH
- L402: renamed from L5; value SRR6038-5R0Y -> 5uH
- Q701: renamed from Q2; value PMOS -> DMP3099L
- R101: renamed from R1; value 10K -> 10kΩ
- R102: renamed from R2; value 470 -> 470Ω
- R103: renamed from R3; value 1k -> 1kΩ
- R104: renamed from R4; value 1k -> 1kΩ
- R105: renamed from R5; value 10K -> 10kΩ
- R106: renamed from R6; value 470 -> 470Ω
- R107: renamed from R7; value 499R -> 499Ω
- R108: renamed from R8; value 3k -> 3kΩ
- R109: renamed from R9; value 18k -> 18kΩ
- R201: renamed from R16; value 10k -> 10kΩ
- R202: renamed from R17; value 14k -> 14kΩ
- R203: renamed from R18; value 56k -> 56kΩ
- R204: renamed from R19; value 10k -> 10kΩ
- R301: renamed from R59; value 10k -> 10kΩ
- R302: renamed from R60; value 113k -> 113kΩ
- R303: renamed from R61; value 10k -> 10kΩ
- R304: renamed from R62; value 2.2 -> 2.2Ω
- R305: renamed from R63; value 1k -> 1kΩ
- R306: renamed from R64; value 442k -> 442kΩ
- R307: renamed from R65; value 200k -> 200kΩ
- R308: renamed from R66; value 100k -> 100kΩ
- R309: renamed from R67; value 10k -> 10kΩ
- R310: renamed from R68; value 5.1R -> 5.1Ω
- R401: renamed from R43; value 7.87k -> 7.87kΩ
- R402: renamed from R44; value 360k -> 360kΩ
- R403: renamed from R45; value 100k -> 100kΩ
- R404: renamed from R46; value 10K -> 10kΩ
- R405: renamed from R47; value 560k -> 560kΩ
- R406: renamed from R48; value 49.9k -> 49.9kΩ
- R407: renamed from R49; value 150k -> 150kΩ
- R408: renamed from R50; value 301k -> 301kΩ
- R409: renamed from R51; value 18.7k -> 18.7kΩ
- R410: renamed from R52; value 976k -> 976kΩ
- R411: renamed from R53; value 100k -> 100kΩ
- R412: renamed from R54; value 49.9k -> 49.9kΩ
- R413: renamed from R55; value 432k -> 432kΩ
- R414: renamed from R56; value 10K -> 10kΩ
- R415: renamed from R57; value 475k -> 475kΩ
- R416: renamed from R58; value 287k -> 287kΩ
- R501: renamed from R10; value 0 -> 0Ω
- R502: renamed from R11; value 60 -> 60Ω
- R503: renamed from R12; value 60 -> 60Ω
- R601: renamed from R13; value 5.1k -> 5.1kΩ
- R602: renamed from R14; value 5.1k -> 5.1kΩ
- R603: renamed from R15; value 5.1k -> 5.1kΩ
- R701: renamed from R69; value 1k -> 1kΩ
- R702: renamed from R70; value 10k -> 10kΩ
- R801: renamed from R21; value 75k -> 75kΩ
- R802: renamed from R22; value 14k -> 14kΩ
- R803: renamed from R23; value 10k -> 10kΩ
- R804: renamed from R24; value 75k -> 75kΩ
- R805: renamed from R25; value 14k -> 14kΩ
- R806: renamed from R26; value 10k -> 10kΩ
- R807: renamed from R27; value 1k -> 1kΩ
- R808: renamed from R28; value 1k -> 1kΩ
- R809: renamed from R29; value 49.9 -> 49.9Ω
- R810: renamed from R30; value 49.9 -> 49.9Ω
- R811: renamed from R31; value 1k -> 1kΩ
- R812: renamed from R32; value 1k -> 1kΩ
- R813: renamed from R33; value 75k -> 75kΩ
- R814: renamed from R34; value 14k -> 14kΩ
- R815: renamed from R35; value 10k -> 10kΩ
- R816: renamed from R36; value 1k -> 1kΩ
- R817: renamed from R37; value 49.9 -> 49.9Ω
- R818: renamed from R38; value 1k -> 1kΩ
- R901: renamed from R39; value 100 -> 100Ω
- R902: renamed from R40; value 100 -> 100Ω
- R903: renamed from R41; value 100 -> 100Ω
- R904: renamed from R42; value 100 -> 100Ω
- moved R106 35.5 mm to (163.7, 69.2)
- moved D104 33.5 mm to (163.6, 70.1), turned to 0 degrees
- moved R102 12.3 mm to (144.6, 80.0)
- moved D1101 12.2 mm to (137.3, 102.2), turned to -90 degrees
- moved TP101 10.3 mm to (146.6, 78.0)
- moved D101 10.3 mm to (145.6, 80.0)
- moved R104 9.74 mm to (140.2, 82.9), turned to -90 degrees
- moved TP102 9.64 mm to (145.4, 82.7)
- moved R103 9.57 mm to (133.8, 82.9), turned to -90 degrees
- moved R107 6.37 mm to (146.7, 80.0), turned to -90 degrees
- moved D102 5.91 mm to (133.8, 84.8), turned to 90 degrees
- moved D103 5.73 mm to (140.2, 84.8), turned to 90 degrees
- moved R501 4.35 mm to (132.7, 79.3), turned to 180 degrees
- moved C501 3.49 mm to (137.2, 86.5)
- moved JP501 3.45 mm to (137.3, 79.1)
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- renumbered C1 to C101, C2 to C102, C4 to C104, C7 to C107, C9 to C109, C12 to C112, C13 to C113, C17 to C201, C18 to C202, C19 to C203, C20 to C204, C21 to C205, C22 to C206, C23 to C207, C65 to C301, C66 to C302, C67 to C303, C68 to C304, C69 to C305, C70 to C306, C71 to C307, C72 to C308, C73 to C309, C75 to C311, C76 to C312, C77 to C313, C78 to C314, C79 to C315, C80 to C316, C81 to C317, C41 to C401, C42 to C402, C43 to C403, C44 to C404, C45 to C405, C46 to C406, C47 to C407, C48 to C408, C49 to C409, C50 to C410, C51 to C411, C52 to C412, C53 to C413, C54 to C414, C55 to C415, C56 to C416, C57 to C417, C58 to C418, C59 to C419, C60 to C420, C61 to C421, C62 to C422, C63 to C423, C64 to C424, C14 to C501, C15 to C502, C16 to C503, C25 to C801, C26 to C802, C27 to C803, C28 to C804, C29 to C805, C83 to C806, C85 to C807, C30 to C808, C84 to C809, D6 to D1001, CR1 to D1101, CR2 to D401, D1 to D501, D2 to D601, H1 to H101, H2 to H102, H3 to H103, H4 to H104, J8 to J1001, JP1 to J101, JP2 to J102, J1 to J103, J2 to J601, J7 to J701, JP3 to JP501, JP16 to JP701, JP4 to JP801, JP5 to JP802, JP6 to JP803, JP7 to JP804, JP8 to JP805, JP9 to JP806, JP10 to JP807, JP11 to JP808, JP12 to JP809, JP13 to JP810, JP14 to JP811, JP15 to JP812, L2 to L102, L3 to L201, L6 to L301, Q1 to Q301, TP1 to TP101, TP2 to TP102, TP5 to TP201, TP6 to TP202, TP7 to TP203, TP8 to TP204, TP3 to TP601, TP4 to TP602, U1 to U101, U3 to U201, U4 to U202, U5 to U203, U8 to U301, IC2 to U401, IC3 to U402, IC4 to U403, IC5 to U404, U2 to U501, IC1 to U801, U6 to U901, U7 to U902, Y1 to Y101
Connections:
- J1101 pad 3: Net-(J3-Pin_3) -> /ServoPWM
- U101 pad 37: /CAN_TX -> /ServoPWM
- U101 pad 38: /CAN_RX -> /SD_DET
- U101 pad 39: /ServoPWM -> /SD_CS
- U101 pad 40: /SD_DET -> /VSPI_MOSI
- U101 pad 41: /SD_CS -> /VSPI_SCLK
- U101 pad 42: /VSPI_MOSI -> /VSPI_MISO
- U101 pad 43: /VSPI_SCLK -> /SD_EN
- U101 pad 47: /VSPI_MISO -> /CAN_RX
- U101 pad 48: /SD_EN -> /CAN_TX
Routing:
- net /ServoPWM: track 46.7 -> 40.2 mm, vias 2 -> 0
- net Net-(J3-Pin_3): track 5.13 -> 0.00 mm
- net /BUCK_EN: track 28.4 -> 23.6 mm
- net RBUS_uC_V: track 34.6 -> 39.4 mm
- net +12V: track 37.8 -> 33.8 mm
- net +5V: track 39.6 -> 36.8 mm
- net GND: track 10.1 -> 7.50 mm, vias 172 -> 213
- net /T_FAULT0: track 21.2 -> 19.1 mm
- net /T_CS0: track 17.8 -> 15.8 mm
- net /CAN_TX: track 18.7 -> 20.7 mm, vias 0 -> 2
- net /CAN_RX: track 14.3 -> 16.2 mm, vias 0 -> 2
- net /BuckPGOOD: track 24.5 -> 22.7 mm
- net /T_CS1: track 23.6 -> 21.7 mm
- net /SD_EN: track 17.6 -> 16.0 mm
- net /SD_DET: track 30.1 -> 31.8 mm
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Other:
- outline, holes or cut-outs redrawn
- board text added: "12V"
- board text added: "3V3"
- board text added: "5V"
- board text added: "BBIN"
- board text added: "BBOUT"
- board text added: "BOOT"
- board text added: "CANRX"
- board text added: "CANTX"
- board text added: "Data+"
- board text added: "Data-"
- board text added: "Designed by Wayne Wang Electronics 2026"
- board text added: "Logic"
- board text added: "RST"
- board text added: "RXD"
- board text added: "TXD"
- board text removed: "3"
- board text removed: "Designed by Wayne Wang 2026"
- board text removed: "J3"
