File: Hardware/Heimdall.kicad_pcb (KiCad board)
At the start: 4 copper layers, 70 x 50 mm, 227 parts, among them J1001 GPIO Breakout, J101 Conn_01x02_Male, J102 Conn_01x02_Male, J103 RBUS, J1101 1053131103, J601 USB_C_Receptacle_USB2.0, J701 ST1W008S4TR2000, J801 1053131103, J802 1053131103, J803 1053131103, J901 1053131102, J902 1053131102, Q301 SSM3K15AMFV,L3F, Q701 DMP3099L, U101 ESP32-S3, U201 LM66200DRLR, U202 MAX77827AEFD+T, U203 SC4215ASTRT, U301 SiC437AED-T1, U401 TPS61089RNRR, U402 AP2205-W5-7, U403 AP2205-W5-7, U404 TPS61089RNRR, U501 SN65HVD230, U801 ADS131M04IRUKR, U901 MAX31856, U902 MAX31856, Y101 R940000171

Commit message: prod files after final final change
Parts:
- R501: footprint Resistor_SMD:R_0603_1608Metric -> Resistor_SMD:R_0402_1005Metric
- TP101, TP102: moved to B.Cu
- moved G*** 33.6 mm to (171.2, 85.8)
- moved R109 14.1 mm to (145.3, 81.9)
- moved LOGO1 14.1 mm to (142.5, 87.7)
- moved C311 8.23 mm to (133.4, 82.2)
- moved R310 8.23 mm to (134.9, 82.2)
- moved C306 7.97 mm to (127.1, 79.0)
- moved C301 7.83 mm to (134.9, 78.1)
- moved R305 7.62 mm to (135.5, 73.8)
- moved R304 7.62 mm to (128.5, 74.8)
- moved R307 7.62 mm to (131.8, 74.8)
- moved C302 7.62 mm to (134.4, 80.3)
- moved C310 7.62 mm to (129.5, 74.8)
- moved Q301 7.62 mm to (134.1, 73.8)
- moved R302 7.62 mm to (134.9, 76.1)
- moved R303 7.62 mm to (134.9, 77.1)
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Routing:
- net /BUCK_EN: track 23.6 -> 16.9 mm, vias 0 -> 2
- net /RXD: track 8.69 -> 2.25 mm, vias 2 -> 1
- net /BuckPGOOD: track 22.7 -> 16.8 mm
- net +6V: track 12.8 -> 16.4 mm, vias 17 -> 14
- net /Buck/SW: track 4.36 -> 0.91 mm
- net /CAN_RX: track 16.2 -> 13.1 mm
- net /CAN+: track 11.2 -> 14.1 mm
- net /ServoPWM: track 40.2 -> 37.4 mm
- net /CAN_TX: track 20.7 -> 18.1 mm
- net /TXD: track 2.55 -> 4.41 mm, vias 0 -> 1
- net VBUS: track 44.6 -> 46.1 mm
- net RBUS_uC_V: track 39.4 -> 40.9 mm
- net /Buck/VDD: track 11.0 -> 9.61 mm, vias 3 -> 2
- net +16.8V: track 10.7 -> 9.62 mm, vias 19 -> 12
- net +3V3: track 42.8 -> 43.3 mm
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- removed copper zone on B.Cu, net +3V3
- removed copper zone on B.Cu, net Net-(U401-SW)
