File: Hardware/Heimdall.kicad_sch (KiCad schematic)
At the start: 40 parts, among them J1 RBUS, U1 ESP32-S3, Y1 R940000171

Commit message: Version 5
Connections:
- net ADS_CLK: now also U1.51 (GPIO45); no longer U1.9 (GPIO4/ADC1_CH3)
- net ADS_CS: now also U1.7 (GPIO2/ADC1_CH1); no longer U1.11 (GPIO6/ADC1_CH5)
- net ADS_DRDY: now also U1.6 (GPIO1/ADC1_CH0); no longer U1.10 (GPIO5/ADC1_CH4)
- net CAN_RX: now also U1.38 (GPIO33)
- net CAN_TX: now also U1.37 (SPICLK_P/GPIO47)
- net HSPI_MISO: now also U1.10 (GPIO5/ADC1_CH4); no longer U1.39 (GPIO34)
- net HSPI_MOSI: now also U1.9 (GPIO4/ADC1_CH3); no longer U1.38 (GPIO33)
- net HSPI_SCLK: now also U1.11 (GPIO6/ADC1_CH5); no longer U1.40 (GPIO35)
- net SD_DET: now also U1.40 (GPIO35); no longer U1.49 (U0TXD/PROG/GPIO43)
- net ServoPWM: now also U1.39 (GPIO34); no longer U1.7 (GPIO2/ADC1_CH1)
- net at R7.2: now also U1.49 (U0TXD/PROG/GPIO43); no longer U1.37 (SPICLK_P/GPIO47)
- no-connect marks 15 -> 13
Other:
- moved on the sheet: R7

Commit message: tiny tweaks and ready to order
Parts:
- C103: renamed from C3; value 0.1uF -> 100nF
- C105: renamed from C5; value 0.1uF -> 100nF
- C106: renamed from C6; value 0.1uF -> 100nF
- C108: renamed from C8; value 0.1uF -> 100nF
- C110: renamed from C10; value 0.1uF -> 100nF
- C111: renamed from C11; value 0.1uF -> 100nF
- D101: renamed from LED1; value GREEN_LED -> LED_GREEN
- D102: renamed from LED2; value GREEN_LED -> LED_GREEN
- D103: renamed from LED3; value ORANGE_LED -> LED_ORANGE
- D104: renamed from LED4; value BLUE_LED -> LED_BLUE
- D105: renamed from LED5; value RED_LED -> LED_RED
- H101: renamed from H1; now left out of the parts list
- H102: renamed from H2; now left out of the parts list
- H103: renamed from H3; now left out of the parts list
- H104: renamed from H4; now left out of the parts list
- J101: renamed from JP1; now left out of the parts list
- J102: renamed from JP2; now left out of the parts list
- L101: renamed from L1; value 2.0nH -> 2nH
- R101: renamed from R1; value 10K -> 10kΩ
- R102: renamed from R2; value 470 -> 470Ω
- R103: renamed from R3; value 1k -> 1kΩ
- R104: renamed from R4; value 1k -> 1kΩ
- R105: renamed from R5; value 10K -> 10kΩ
- R106: renamed from R6; value 470 -> 470Ω
- R107: renamed from R7; value 499R -> 499Ω
- R108: renamed from R8; value 3k -> 3kΩ
- R109: renamed from R9; value 18k -> 18kΩ
- TP101: renamed from TP1; now left out of the parts list
- TP102: renamed from TP2; now left out of the parts list
- renumbered C1 to C101, C2 to C102, C4 to C104, C7 to C107, C9 to C109, C12 to C112, C13 to C113, J1 to J103, L2 to L102, U1 to U101, Y1 to Y101
Connections:
- net CAN_RX: now also U101.47 (MTDI/JTAG/GPIO41); no longer U101.38 (GPIO33)
- net CAN_TX: now also U101.48 (MTMS/JTAG/GPIO42); no longer U101.37 (SPICLK_P/GPIO47)
- net SD_CS: now also U101.39 (GPIO34); no longer U101.41 (GPIO36)
- net SD_DET: now also U101.38 (GPIO33); no longer U101.40 (GPIO35)
- net SD_EN: now also U101.43 (GPIO38); no longer U101.48 (MTMS/JTAG/GPIO42)
- net ServoPWM: now also U101.37 (SPICLK_P/GPIO47); no longer U101.39 (GPIO34)
- net VSPI_MISO: now also U101.42 (GPIO37); no longer U101.47 (MTDI/JTAG/GPIO41)
- net VSPI_MOSI: now also U101.40 (GPIO35); no longer U101.42 (GPIO37)
- net VSPI_SCLK: now also U101.41 (GPIO36); no longer U101.43 (GPIO38)
