File: Hardware/Sensor_Power.kicad_sch (KiCad schematic)
At the start: 47 parts, among them IC2 TPS61089RNRR, IC3 AP2205-W5-7, IC4 AP2205-W5-7, IC5 TPS61089RNRR

Commit message: tiny tweaks and ready to order
Parts:
- L401: renamed from L4; value SRR6038-5R0Y -> 5uH
- L402: renamed from L5; value SRR6038-5R0Y -> 5uH
- R401: renamed from R43; value 7.87k -> 7.87kΩ
- R402: renamed from R44; value 360k -> 360kΩ
- R403: renamed from R45; value 100k -> 100kΩ
- R404: renamed from R46; value 10K -> 10kΩ
- R405: renamed from R47; value 560k -> 560kΩ
- R406: renamed from R48; value 49.9k -> 49.9kΩ
- R407: renamed from R49; value 150k -> 150kΩ
- R408: renamed from R50; value 301k -> 301kΩ
- R409: renamed from R51; value 18.7k -> 18.7kΩ
- R410: renamed from R52; value 976k -> 976kΩ
- R411: renamed from R53; value 100k -> 100kΩ
- R412: renamed from R54; value 49.9k -> 49.9kΩ
- R413: renamed from R55; value 432k -> 432kΩ
- R414: renamed from R56; value 10K -> 10kΩ
- R415: renamed from R57; value 475k -> 475kΩ
- R416: renamed from R58; value 287k -> 287kΩ
- renumbered C41 to C401, C42 to C402, C43 to C403, C44 to C404, C45 to C405, C46 to C406, C47 to C407, C48 to C408, C49 to C409, C50 to C410, C51 to C411, C52 to C412, C53 to C413, C54 to C414, C55 to C415, C56 to C416, C57 to C417, C58 to C418, C59 to C419, C60 to C420, C61 to C421, C62 to C422, C63 to C423, C64 to C424, CR2 to D401, IC2 to U401, IC3 to U402, IC4 to U403, IC5 to U404
