File: Hardware/sd.kicad_sch (KiCad schematic)
At the start: 6 parts, among them J7 ST1W008S4TR2000, Q2 PMOS

Commit message: tiny tweaks and ready to order
Parts:
- C701: renamed from C82; value 0.1uF -> 100nF
- JP701: renamed from JP16; now left out of the parts list
- Q701: renamed from Q2; value PMOS -> DMP3099L
- R701: renamed from R69; value 1k -> 1kΩ
- R702: renamed from R70; value 10k -> 10kΩ
- renumbered J7 to J701
Other:
- moved on the sheet: JP701
Changed lines of the file:
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@@
 	(wire
 		(pts
-			(xy 78.74 69.85) (xy 78.74 72.39)
+			(xy 73.66 69.85) (xy 73.66 72.39)
 		)
 		(stroke
@@
 	(wire
 		(pts
-			(xy 78.74 62.23) (xy 78.74 58.42)
+			(xy 73.66 62.23) (xy 73.66 58.42)
 		)
 		(stroke
@@
 	(wire
 		(pts
-			(xy 78.74 58.42) (xy 90.17 58.42)
+			(xy 73.66 58.42) (xy 90.17 58.42)
 		)
 		(stroke
@@
 	(wire
 		(pts
-			(xy 78.74 72.39) (xy 90.17 72.39)
+			(xy 73.66 72.39) (xy 90.17 72.39)
 		)
 		(stroke
@@
 		(on_board yes)
 		(dnp no)
-		(property "Reference" "#PWR0145"
+		(property "Reference" "#PWR0703"
 			(at 100.33 82.55 0)
 			(effects
@@
 		)
 		(instances
-			(project "Reggie"
+			(project "Heimdall"
 				(path "/7db990e4-92e1-4f99-b4d2-435bbec1ba83/b3c2f461-38d3-4d4d-a4e6-b155780b2822"
-					(reference "#PWR0145")
+					(reference "#PWR0703")
 					(unit 1)
 				)
@@
 		(on_board yes)
 		(dnp no)
-		(property "Reference" "C82"
+		(property "Reference" "C701"
 			(at 85.09 87.0966 90)
 			(effects
@@
 			)
 		)
-		(property "Value" "0.1uF"
+		(property "Value" "100nF"
 			(at 85.09 89.408 90)
 			(effects
@@
 		)
 		(instances
-			(project "RicardoTemplate"
+			(project "Heimdall"
 				(path "/7db990e4-92e1-4f99-b4d2-435bbec1ba83/b3c2f461-38d3-4d4d-a4e6-b155780b2822"
-					(reference "C82")
+					(reference "C701")
 					(unit 1)
 				)
@@
 		(on_board yes)
 		(dnp no)
-		(property "Reference" "#PWR0144"
+		(property "Reference" "#PWR0704"
 			(at 105.41 96.52 0)
 			(effects
@@
 		)
 		(instances
-			(project "RicardoTemplate"
+			(project "Heimdall"
 				(path "/7db990e4-92e1-4f99-b4d2-435bbec1ba83/b3c2f461-38d3-4d4d-a4e6-b155780b2822"
-					(reference "#PWR0144")
+					(reference "#PWR0704")
 					(unit 1)
 				)
@@
 		(on_board yes)
 		(dnp no)
-		(property "Reference" "#PWR0146"
+		(property "Reference" "#PWR0705"
 			(at 124.46 62.484 0)
 			(effects
@@
 		)
 		(instances
-			(project "RicardoTemplate"
+			(project "Heimdall"
 				(path "/7db990e4-92e1-4f99-b4d2-435bbec1ba83/b3c2f461-38d3-4d4d-a4e6-b155780b2822"
-					(reference "#PWR0146")
+					(reference "#PWR0705")
 					(unit 1)
 				)
@@
 		(dnp no)
 		(fields_autoplaced yes)
-		(property "Reference" "#PWR0143"
+		(property "Reference" "#PWR0702"
 			(at 90.17 55.88 0)
 			(effects
@@
 		)
 		(instances
-			(project "RicardoTemplate"
+			(project "Heimdall"
 				(path "/7db990e4-92e1-4f99-b4d2-435bbec1ba83/b3c2f461-38d3-4d4d-a4e6-b155780b2822"
-					(reference "#PWR0143")
+					(reference "#PWR0702")
 					(unit 1)
 				)
@@
 		(on_board yes)
 		(dnp no)
-		(property "Reference" "R70"
+		(property "Reference" "R702"
 			(at 120.65 60.96 0)
 			(effects
@@
 			)
 		)
-		(property "Value" "10k"
+		(property "Value" "10kΩ"
 			(at 120.65 63.5 0)
 			(effects
@@
 		)
 		(instances
-			(project "RicardoTemplate"
+			(project "Heimdall"
 				(path "/7db990e4-92e1-4f99-b4d2-435bbec1ba83/b3c2f461-38d3-4d4d-a4e6-b155780b2822"
-					(reference "R70")
+					(reference "R702")
 					(unit 1)
 				)
@@
 		(dnp no)
 		(fields_autoplaced yes)
-		(property "Reference" "Q2"
-			(at 86.36 64.77 0)
+		(property "Reference" "Q701"
+			(at 86.36 64.7699 0)
 			(effects
 				(font
@@
 			)
 		)
-		(property "Value" "PMOS"
-			(at 86.36 67.31 0)
+		(property "Value" "DMP3099L"
+			(at 86.36 67.3099 0)
 			(effects
 				(font
@@
 		)
 		(instances
-			(project "Reggie"
+			(project "Heimdall"
 				(path "/7db990e4-92e1-4f99-b4d2-435bbec1ba83/b3c2f461-38d3-4d4d-a4e6-b155780b2822"
-					(reference "Q2")
+					(reference "Q701")
 					(unit 1)
 				)
@@
 		(dnp no)
 		(fields_autoplaced yes)
-		(property "Reference" "J7"
+		(property "Reference" "J701"
 			(at 138.43 64.4355 0)
 			(effects
@@
 		)
 		(instances
-			(project "RicardoTemplate"
+			(project "Heimdall"
 				(path "/7db990e4-92e1-4f99-b4d2-435bbec1ba83/b3c2f461-38d3-4d4d-a4e6-b155780b2822"
-					(reference "J7")
+					(reference "J701")
 					(unit 1)
 				)
@@
 	(symbol
 		(lib_id "Jumper:SolderJumper_2_Open")
-		(at 78.74 66.04 270)
+		(at 73.66 66.04 270)
 		(unit 1)
 		(exclude_from_sim no)
-		(in_bom yes)
+		(in_bom no)
 		(on_board yes)
 		(dnp no)
-		(property "Reference" "JP16"
+		(property "Reference" "JP701"
+			(at 68.58 66.04 90)
+			(effects
+				(font
+					(size 1.27 1.27)
+				)
+			)
+		)
+		(property "Value" "SolderJumper_2_Open"
+			(at 41.91 48.26 0)
+			(effects
+				(font
+					(size 1.27 1.27)
+				)
+				(hide yes)
+			)
+		)
+		(property "Footprint" "iclr:SmallerSolderJP"
 			(at 73.66 66.04 0)
 			(effects
@@
 					(size 1.27 1.27)
 				)
-			)
-		)
-		(property "Value" "SolderJumper_2_Open"
-			(at 46.99 48.26 0)
-			(effects
-				(font
-					(size 1.27 1.27)
-				)
-				(hide yes)
-			)
-		)
-		(property "Footprint" "iclr:SmallerSolderJP"
-			(at 78.74 66.04 0)
-			(effects
-				(font
-					(size 1.27 1.27)
-				)
 				(hide yes)
 			)
 		)
 		(property "Datasheet" "~"
-			(at 78.74 66.04 0)
+			(at 73.66 66.04 0)
 			(effects
 				(font
@@
 		)
 		(property "Description" ""
-			(at 78.74 66.04 0)
+			(at 73.66 66.04 0)
 			(effects
 				(font
@@
 		)
 		(instances
-			(project "Reggie"
+			(project "Heimdall"
 				(path "/7db990e4-92e1-4f99-b4d2-435bbec1ba83/b3c2f461-38d3-4d4d-a4e6-b155780b2822"
-					(reference "JP16")
+					(reference "JP701")
 					(unit 1)
 				)
@@
 		(on_board yes)
 		(dnp no)
-		(property "Reference" "R69"
+		(property "Reference" "R701"
 			(at 96.901 71.2501 0)
 			(effects
@@
 			)
 		)
-		(property "Value" "1k"
+		(property "Value" "1kΩ"
 			(at 96.901 73.787 0)
 			(effects
@@
 		)
 		(instances
-			(project "Reggie"
+			(project "Heimdall"
 				(path "/7db990e4-92e1-4f99-b4d2-435bbec1ba83/b3c2f461-38d3-4d4d-a4e6-b155780b2822"
-					(reference "R69")
+					(reference "R701")
 					(unit 1)
 				)
@@
 		(dnp no)
 		(fields_autoplaced yes)
-		(property "Reference" "#PWR0147"
+		(property "Reference" "#PWR0706"
 			(at 152.4 109.22 0)
 			(effects
@@
 		)
 		(instances
-			(project "RicardoTemplate"
+			(project "Heimdall"
 				(path "/7db990e4-92e1-4f99-b4d2-435bbec1ba83/b3c2f461-38d3-4d4d-a4e6-b155780b2822"
-					(reference "#PWR0147")
+					(reference "#PWR0706")
 					(unit 1)
 				)
@@
 		(on_board yes)
 		(dnp no)
-		(property "Reference" "#PWR0142"
+		(property "Reference" "#PWR0701"
 			(at 80.01 90.17 0)
 			(effects
@@
 		)
 		(instances
-			(project "RicardoTemplate"
+			(project "Heimdall"
 				(path "/7db990e4-92e1-4f99-b4d2-435bbec1ba83/b3c2f461-38d3-4d4d-a4e6-b155780b2822"
-					(reference "#PWR0142")
+					(reference "#PWR0701")
 					(unit 1)
 				)
